Commit message: adicionando world

File: src/my_bot/description/lidar.xacro (robot description, xacro)
@@ -7,4 +7,48 @@
     </joint>
     <link name="laser_frame">
+         <visual>
+            <geometry>
+                <cylinder radius="0.05" length="0.04"/>
+            </geometry>
+            <material name="red"/>
+        </visual>
+        <collision>
+            <geometry>
+                <cylinder radius="0.05" length="0.04"/>
+            </geometry>
+        </collision>
+        <xacro:inertial_cylinder mass="0.1" length="0.04" radius="0.05">
+            <origin xyz="0 0 0" rpy="0 0 0"/>
+        </xacro:inertial_cylinder>
     </link>
+    <gazebo reference="laser_frame">
+        <material>Gazebo/Red</material>
+        <sensor name="laser" type="ray">
+            <pose> 0 0 0 0 0 0 </pose>
+            <visualize>true</visualize>
+            <update_rate>10</update_rate>
+            <ray>
+                <scan>
+                    <horizontal>
+                        <samples>360</samples>
+                        <resolution>1</resolution>
+                        <min_angle>-3.14</min_angle>
+                        <max_angle>3.14</max_angle>
+                    </horizontal>
+                </scan>
+                <range>
+                    <min>0.3</min>
+                    <max>12</max>
+                    <resolution>0.01</resolution>
+                </range>
+            </ray>
+            <plugin name="laser_controller" filename="libgazebo_ros_ray_sensor.so">
+                <ros>
+                    <argument>~/out:=scan</argument>
+                </ros>
+                <output_type>sensor_msgs/LaserScan</output_type>
+                <frame_name>laser_frame</frame_name>
+            </plugin>
+        </sensor>
+    </gazebo>
 </robot>

Commit message: adicionando meu mundo de obstaculos

File: src/my_bot/description/lidar.xacro (robot description, xacro)
@@ -23,9 +23,9 @@
     </link>
     <gazebo reference="laser_frame">
-        <material>Gazebo/Red</material>
-        <sensor name="laser" type="ray">
-            <pose> 0 0 0 0 0 0 </pose>
+        <sensor name="laser" type="gpu_ray">
+            <always_on>true</always_on>
             <visualize>true</visualize>
             <update_rate>10</update_rate>
+            <topic>scan</topic>
             <ray>
                 <scan>
@@ -39,14 +39,10 @@
                 <range>
                     <min>0.3</min>
-                    <max>12</max>
-                    <resolution>0.01</resolution>
+                    <max>12.0</max>
                 </range>
             </ray>
-            <plugin name="laser_controller" filename="libgazebo_ros_ray_sensor.so">
-                <ros>
-                    <argument>~/out:=scan</argument>
-                </ros>
-                <output_type>sensor_msgs/LaserScan</output_type>
-                <frame_name>laser_frame</frame_name>
+            <plugin filename="libignition-gazebo-sensors-system.so"
+                    name="ignition::gazebo::systems::Sensors">
+                <render_engine>ogre2</render_engine>
             </plugin>
         </sensor>

Commit message: corrigindo lidar na odom

File: src/my_bot/description/lidar.xacro (robot description, xacro)
@@ -7,5 +7,5 @@
     </joint>
     <link name="laser_frame">
-         <visual>
+        <visual>
             <geometry>
                 <cylinder radius="0.05" length="0.04"/>
@@ -23,16 +23,17 @@
     </link>
     <gazebo reference="laser_frame">
-        <sensor name="laser" type="gpu_ray">
+        <sensor name="laser" type="gpu_lidar">   <!-- era gpu_ray -->
             <always_on>true</always_on>
             <visualize>true</visualize>
             <update_rate>10</update_rate>
             <topic>scan</topic>
-            <ray>
+            <gz_frame_id>laser_frame</gz_frame_id>  <!-- ✅ necessário para o TF -->
+            <lidar>                                  <!-- ✅ era <ray> -->
                 <scan>
                     <horizontal>
-                        <samples>360</samples>
+                        <samples>1</samples>
                         <resolution>1</resolution>
-                        <min_angle>-3.14</min_angle>
-                        <max_angle>3.14</max_angle>
+                        <min_angle>0</min_angle>
+                        <max_angle>0</max_angle>
                     </horizontal>
                 </scan>
@@ -41,7 +42,7 @@
                     <max>12.0</max>
                 </range>
-            </ray>
-            <plugin filename="libignition-gazebo-sensors-system.so"
-                    name="ignition::gazebo::systems::Sensors">
+            </lidar>
+            <plugin filename="gz-sim-sensors-system"
+                    name="gz::sim::systems::Sensors">
                 <render_engine>ogre2</render_engine>
             </plugin>
